File: keyboard-pcb.kicad_pcb (KiCad board)
At the start: 2 copper layers, 198 parts, among them J1 Conn_01x04, J3 USB_C_Receptacle_USB2.0_16P, J4 Conn_01x05, SW1 SW_Push, SW2 SW_Push, U1 RP2040, U2 XC6206PxxxMR, U3 W25Q128JVS, U5 SRV05-4, Y1 Crystal_GND24_Small

Commit message: Wired components of PCB
Type-C 2.0 Connector system
Parts:
- removed SW2: SW_Push, Button_Switch_SMD:SW_SPST_TL3342
- added BOOT1: SW_Push, Button_Switch_SMD:SW_SPST_TL3342, B.Cu at (157.2, 164.3)
- added C13: 100nF, Capacitor_SMD:C_0402_1005Metric, B.Cu at (147.6, 183.3)
- added C14: 100nF, Capacitor_SMD:C_0402_1005Metric, B.Cu at (143.4, 183.3)
- added C15: 100nF, Capacitor_SMD:C_0402_1005Metric, B.Cu at (146.6, 183.3)
- added C16: 100nF, Capacitor_SMD:C_0402_1005Metric, B.Cu at (147.2, 194.4)
- C1, C10, C11, C12, C2, C4, C5, C6, C7, C8, C9: footprint Capacitor_SMD:C_0805_2012Metric -> Capacitor_SMD:C_0402_1005Metric
- C3: footprint Capacitor_SMD:C_0805_2012Metric -> Capacitor_SMD:C_0603_1608Metric
- R1, R2, R3, R4, R5, R6, R7, R8, R9: footprint Resistor_SMD:R_0805_2012Metric -> Resistor_SMD:R_0402_1005Metric
- moved J1 175.7 mm to (66.7, 100.4), turned to -90 degrees
- moved J3 175.3 mm to (66.7, 82.5), turned to 0 degrees
- moved F1 161.9 mm to (60.3, 94.3), turned to -90 degrees
- moved R2 158.8 mm to (63.8, 89.7)
- moved U5 156.7 mm to (66.9, 93.0)
- moved R1 153.1 mm to (69.8, 89.7), turned to 0 degrees
- moved U3 73.2 mm to (157.2, 179.4), turned to -90 degrees
- moved C2 69.5 mm to (131.0, 161.9)
- moved R9 66.3 mm to (150.9, 161.7)
- moved R8 64.7 mm to (150.9, 160.3)
- moved C1 62.2 mm to (135.8, 164.7), turned to 90 degrees
- moved R7 58.7 mm to (150.9, 163.5)
- moved U2 57.0 mm to (132.6, 165.1)
- moved C3 51.6 mm to (138.9, 181.0)
- moved C4 50.0 mm to (144.5, 183.3), turned to 90 degrees
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Connections:
- D1 pad 1: col17 -> row0
- D10 pad 1: col17 -> row0
- D11 pad 1: col17 -> row0
- D12 pad 1: col17 -> row0
- D13 pad 1: col17 -> row0
- D2 pad 1: col17 -> row0
- D3 pad 1: col17 -> row0
- D4 pad 1: col17 -> row0
- D5 pad 1: col17 -> row0
- D6 pad 1: col17 -> row0
- D7 pad 1: col17 -> row0
- D8 pad 1: col17 -> row0
- D9 pad 1: col17 -> row0
Routing:
- net D+: track 0.00 -> 199.7 mm
- net D-: track 0.00 -> 196.8 mm
- net +5V: track 0.00 -> 153.1 mm
- net GND: track 0.00 -> 88.3 mm, vias 0 -> 8
- net +3V3: track 0.00 -> 38.9 mm
- net VBUS: track 0.00 -> 16.0 mm
- net Net-(U1-USB_DP): track 0.00 -> 5.31 mm
- net Net-(U1-USB_DM): track 0.00 -> 5.30 mm
- net +1V1: track 0.00 -> 3.87 mm
- net Net-(J3-CC1): track 0.00 -> 3.57 mm
- net Net-(J3-CC2): track 0.00 -> 3.48 mm
- added copper zone on B.Cu, net GND
- added copper zone on F.Cu, net GND
Other:
- board outline added: 357.2 x 135.7 mm
